File: PiBreak.sch (KiCad schematic (older format))
At the start: 6 parts, among them P1 RASPBERRY_PI_P1, P2 CONN_17, P3 CONN_8, P4 CONN_8, P5 CONN_8, P6 CONN_4X2

Commit message: Bump version to 1.0
Parts:
- removed P1: RASPBERRY_PI_P1, symbol RASPBERRY_PI_P1
- removed P2: CONN_17, ~, symbol CONN_17
- removed P6: CONN_4X2, ~, symbol CONN_4X2
- added P1: RASPBERRY_PI_PLUS_CON, symbol RASPBERRY_PI_PLUS_CON
- added P2: CONN_20, symbol CONN_20
- added P3: CONN_6, symbol CONN_6
- added P7: CONN_2, symbol CONN_2
- renumbered P3 to P4, P4 to P5, P5 to P6
Connections:
- net labels added: EEPROM_SCL, EEPROM_SDA, GPIO12, GPIO13, GPIO16, GPIO19, GPIO20, GPIO21, GPIO26, GPIO5, GPIO6
- net labels removed: 3V3, 5V
- wire segments 53 -> 65
- no-connect marks 8 -> 0
Other:
- note added: "Raspberry Pi B+ Connector"
- note removed: "NB: Not broken out on PCB, empty pads only."
- note removed: "NB: On Rev 1 Pi\nPin 3 = GPIO 0\nPin 5 = GPIO 1\nPin 13 = GPIO 21"
- note removed: "Raspberry Pi P1 Connector"
- note removed: "Raspberry Pi P5 Connector"
- moved on the sheet: P4, P5, P6
